File: phase90plusplus.kicad_sch (KiCad schematic)
At the start: 14 parts

Commit message: Hardware commit.
Parts:
- removed J?: AudioJack2, symbol Connector:AudioJack2
- added C10, C4, C6, C8, C9: 47n, symbol Device:C_Small
- added C5: 15u, Capacitor_THT:CP_Radial_D4.0mm_P1.50mm, symbol Device:C_Polarized_Small
- added C7: 0.01u, symbol Device:C_Small
- added J?: AudioJack3, symbol Connector:AudioJack3
- added J?: Barrel_Jack_Switch, symbol Connector:Barrel_Jack_Switch
- added Q1, Q2, Q3, Q4: 2N7000, Package_TO_SOT_THT:TO-92_Inline, symbol Transistor_FET:2N7000
- added Q5: 2N2219, Package_TO_SOT_THT:TO-39-3, symbol Transistor_BJT:2N2219
- added R10, R16, R19, R6: 24K, Resistor_THT:R_Axial_DIN0207_L6.3mm_D2.5mm_P10.16mm_Horizontal, symbol Device:R_Small_US
- added R11, R12, R21, R22, R23: 150K, Resistor_THT:R_Axial_DIN0207_L6.3mm_D2.5mm_P10.16mm_Horizontal, symbol Device:R_Small_US
- added R13, R15, R17, R18, R20, R5, R7, R9: 10K, Resistor_THT:R_Axial_DIN0207_L6.3mm_D2.5mm_P10.16mm_Horizontal, symbol Device:R_Small_US
- added R14: 470K, Resistor_THT:R_Axial_DIN0207_L6.3mm_D2.5mm_P10.16mm_Horizontal, symbol Device:R_Small_US
- added R24: 56K, Resistor_THT:R_Axial_DIN0207_L6.3mm_D2.5mm_P10.16mm_Horizontal, symbol Device:R_Small_US
- added R25: 150k, Resistor_THT:R_Axial_DIN0207_L6.3mm_D2.5mm_P10.16mm_Horizontal, symbol Device:R_Small_US
- added R8: 3M9, Resistor_THT:R_Axial_DIN0207_L6.3mm_D2.5mm_P10.16mm_Horizontal, symbol Device:R_Small_US
- added RV2: 470K, symbol Device:R_Potentiometer_US
- added SW1: SW_SPDT, symbol Switch:SW_SPDT
- added U2, U3, U4, U5, U6: TL061, Package_DIP:DIP-8_W7.62mm, symbol Amplifier_Operational:TL061
- BT1: renamed from BT?; footprint (none) -> Connector_JST:JST_ACH_BM04B-ACHSS-A-GAN-ETF_1x04-1MP_P1.20mm_Vertical
- C1: renamed from C?; footprint (none) -> Capacitor_THT:CP_Radial_D4.0mm_P1.50mm
- R1, R4: renamed from R?; footprint (none) -> Resistor_THT:R_Axial_DIN0207_L6.3mm_D2.5mm_P10.16mm_Horizontal
- R2: renamed from R?; value 10K -> 500k; footprint (none) -> Resistor_THT:R_Axial_DIN0207_L6.3mm_D2.5mm_P10.16mm_Horizontal
- R3: renamed from R?; value 470K -> 500k; footprint (none) -> Resistor_THT:R_Axial_DIN0207_L6.3mm_D2.5mm_P10.16mm_Horizontal
- U1: renamed from U?; footprint (none) -> Package_DIP:DIP-8_W7.62mm
- gave numbers to parts that had none: 6
Connections:
- net +5V: now also Q1.3 (D), Q2.3 (D), Q3.3 (D), Q4.3 (D), Q5.3 (C), R10.1, R12.2, R16.1, R19.1, R6.1
- net +9V: now also U2.7 (V+), U3.7 (V+), U4.7 (V+), U5.7 (V+), U6.7 (V+); no longer BT1.1 (+)
- net GNDREF: now also J2.T, C5.2, J?.R, R24.1, R25.1, U2.4 (V-), U3.4 (V-), U4.4 (V-), U5.4 (V-), U6.4 (V-); no longer BT1.2 (-)
- net VDD: now also Q1.2 (G), Q2.2 (G), Q3.2 (G), Q4.2 (G), R8.2
- net OUTPUT: now reaches J2.S
- net OUTPUT: now also C10.2, R25.2, SW1.3 (C)
- net U1_LOOPBACK: now reaches U1.2 (-), U1.6
- net U1_LOOPBACK: now also C4.1, R22.1, R5.1
- net at R2.1: now also SW1.1 (A)
- new net: R15.2, R17.1, U5.2 (-)
- new net: C9.1, R17.2, R18.1, U5.6
- new net: C10.1, Q5.1 (E), R23.2, R24.2
- new net: C6.2, Q2.1 (S), R10.2, U3.3 (+)
- new net: C9.2, Q4.1 (S), R19.2, U6.3 (+)
- new net: R13.1, R9.2, U3.2 (-)
- new net: C8.1, R13.2, R15.1, U3.6
- new net: J?.T, SW1.2 (B)
- new net: R12.1, R14.2, U4.3 (+)
- new net: R18.2, R20.1, U6.2 (-)
- new net: R20.2, R21.1, U6.6
- new net: C6.1, R7.2, R9.1, U2.6
- new net: C7.1, R11.1, U4.2 (-)
- new net: C5.1, R11.2, R8.1, RV2.1, RV2.2
- new net: C7.2, R14.1, RV2.3, U4.6
- new net: C8.2, Q3.1 (S), R16.2, U5.3 (+)
- new net: R5.2, R7.1, U2.2 (-)
- new net: C4.2, Q1.1 (S), R6.2, U2.3 (+)
- new net: Q5.2 (B), R21.2, R22.2, R23.1
- new net SLEEVE: BT1.2 (-), J?.S
- no-connect marks 2 -> 12
Other:
- note added: "TODO: ADD POLARITY PROTECTION, MAYBE AN INDICATOR LED ALSO FIX THE BATTERY SWITCHING CIRCUIT"
- moved on the sheet: BT1, J2

Commit message: Added libraries, initial routing and layout started.  Schematic revised to add LED and power handling.
Parts:
- removed J2: AudioJack2, symbol Connector:AudioJack2
- removed SW1: SW_SPDT, symbol Switch:SW_SPDT
- added D3: 1N914, Diode_THT:D_DO-35_SOD27_P7.62mm_Horizontal, symbol Diode:1N914
- added D4: LED, LED_THT:LED_D3.0mm, symbol Device:LED
- added J3: AudioJack3, Connector_Audio:Jack_6.35mm_Neutrik_NRJ6HM-1_Horizontal, symbol Connector:AudioJack3
- added R5: 370, Resistor_THT:R_Axial_DIN0207_L6.3mm_D2.5mm_P7.62mm_Horizontal, symbol Device:R_Small_US
- added S1: SWITCH-3PDT-PTH-STOMP, Switches:STOMP_SWITCH_3PDT, symbol SparkFun-Switches:SWITCH-3PDT-PTH-STOMP
- BT1: footprint Connector_JST:JST_ACH_BM04B-ACHSS-A-GAN-ETF_1x04-1MP_P1.20mm_Vertical -> Connector_JST:JST_ACH_BM02B-ACHSS-GAN-ETF_1x02-1MP_P1.20mm_Vertical
- C10, C2, C3, C4, C6, C7, C8, C9: footprint (none) -> Capacitor_THT:C_Disc_D7.5mm_W2.5mm_P5.00mm
- J1: renamed from J?; footprint (none) -> Connector_Audio:Jack_6.35mm_Neutrik_NRJ6HM-1_Horizontal
- J2: renamed from J?; footprint (none) -> Connector_BarrelJack:BarrelJack_Horizontal
- Q5: footprint Package_TO_SOT_THT:TO-39-3 -> Package_TO_SOT_THT:TO-92_Inline
- R1, R2, R3, R4: footprint Resistor_THT:R_Axial_DIN0207_L6.3mm_D2.5mm_P10.16mm_Horizontal -> Resistor_THT:R_Axial_DIN0207_L6.3mm_D2.5mm_P7.62mm_Horizontal
- R10: renamed from R9; footprint Resistor_THT:R_Axial_DIN0207_L6.3mm_D2.5mm_P10.16mm_Horizontal -> Resistor_THT:R_Axial_DIN0207_L6.3mm_D2.5mm_P7.62mm_Horizontal
- R11: renamed from R10; footprint Resistor_THT:R_Axial_DIN0207_L6.3mm_D2.5mm_P10.16mm_Horizontal -> Resistor_THT:R_Axial_DIN0207_L6.3mm_D2.5mm_P7.62mm_Horizontal
- R12: renamed from R11; footprint Resistor_THT:R_Axial_DIN0207_L6.3mm_D2.5mm_P10.16mm_Horizontal -> Resistor_THT:R_Axial_DIN0207_L6.3mm_D2.5mm_P7.62mm_Horizontal
- R13: renamed from R12; footprint Resistor_THT:R_Axial_DIN0207_L6.3mm_D2.5mm_P10.16mm_Horizontal -> Resistor_THT:R_Axial_DIN0207_L6.3mm_D2.5mm_P7.62mm_Horizontal
- R14: renamed from R13; footprint Resistor_THT:R_Axial_DIN0207_L6.3mm_D2.5mm_P10.16mm_Horizontal -> Resistor_THT:R_Axial_DIN0207_L6.3mm_D2.5mm_P7.62mm_Horizontal
- R15: renamed from R14; footprint Resistor_THT:R_Axial_DIN0207_L6.3mm_D2.5mm_P10.16mm_Horizontal -> Resistor_THT:R_Axial_DIN0207_L6.3mm_D2.5mm_P7.62mm_Horizontal
- R16: renamed from R15; footprint Resistor_THT:R_Axial_DIN0207_L6.3mm_D2.5mm_P10.16mm_Horizontal -> Resistor_THT:R_Axial_DIN0207_L6.3mm_D2.5mm_P7.62mm_Horizontal
- R17: renamed from R16; footprint Resistor_THT:R_Axial_DIN0207_L6.3mm_D2.5mm_P10.16mm_Horizontal -> Resistor_THT:R_Axial_DIN0207_L6.3mm_D2.5mm_P7.62mm_Horizontal
- R18: renamed from R17; footprint Resistor_THT:R_Axial_DIN0207_L6.3mm_D2.5mm_P10.16mm_Horizontal -> Resistor_THT:R_Axial_DIN0207_L6.3mm_D2.5mm_P7.62mm_Horizontal
- R19: renamed from R18; footprint Resistor_THT:R_Axial_DIN0207_L6.3mm_D2.5mm_P10.16mm_Horizontal -> Resistor_THT:R_Axial_DIN0207_L6.3mm_D2.5mm_P7.62mm_Horizontal
- R20: renamed from R19; footprint Resistor_THT:R_Axial_DIN0207_L6.3mm_D2.5mm_P10.16mm_Horizontal -> Resistor_THT:R_Axial_DIN0207_L6.3mm_D2.5mm_P7.62mm_Horizontal
- R21: renamed from R20; footprint Resistor_THT:R_Axial_DIN0207_L6.3mm_D2.5mm_P10.16mm_Horizontal -> Resistor_THT:R_Axial_DIN0207_L6.3mm_D2.5mm_P7.62mm_Horizontal
- R22: renamed from R21; footprint Resistor_THT:R_Axial_DIN0207_L6.3mm_D2.5mm_P10.16mm_Horizontal -> Resistor_THT:R_Axial_DIN0207_L6.3mm_D2.5mm_P7.62mm_Horizontal
- R23: renamed from R22; footprint Resistor_THT:R_Axial_DIN0207_L6.3mm_D2.5mm_P10.16mm_Horizontal -> Resistor_THT:R_Axial_DIN0207_L6.3mm_D2.5mm_P7.62mm_Horizontal
- R24: renamed from R23; footprint Resistor_THT:R_Axial_DIN0207_L6.3mm_D2.5mm_P10.16mm_Horizontal -> Resistor_THT:R_Axial_DIN0207_L6.3mm_D2.5mm_P7.62mm_Horizontal
- R25: renamed from R24; footprint Resistor_THT:R_Axial_DIN0207_L6.3mm_D2.5mm_P10.16mm_Horizontal -> Resistor_THT:R_Axial_DIN0207_L6.3mm_D2.5mm_P7.62mm_Horizontal
- R26: renamed from R25; footprint Resistor_THT:R_Axial_DIN0207_L6.3mm_D2.5mm_P10.16mm_Horizontal -> Resistor_THT:R_Axial_DIN0207_L6.3mm_D2.5mm_P7.62mm_Horizontal
- R6: renamed from R5; footprint Resistor_THT:R_Axial_DIN0207_L6.3mm_D2.5mm_P10.16mm_Horizontal -> Resistor_THT:R_Axial_DIN0207_L6.3mm_D2.5mm_P7.62mm_Horizontal
- R7: renamed from R6; footprint Resistor_THT:R_Axial_DIN0207_L6.3mm_D2.5mm_P10.16mm_Horizontal -> Resistor_THT:R_Axial_DIN0207_L6.3mm_D2.5mm_P7.62mm_Horizontal
- R8: renamed from R7; footprint Resistor_THT:R_Axial_DIN0207_L6.3mm_D2.5mm_P10.16mm_Horizontal -> Resistor_THT:R_Axial_DIN0207_L6.3mm_D2.5mm_P7.62mm_Horizontal
- R9: renamed from R8; footprint Resistor_THT:R_Axial_DIN0207_L6.3mm_D2.5mm_P10.16mm_Horizontal -> Resistor_THT:R_Axial_DIN0207_L6.3mm_D2.5mm_P7.62mm_Horizontal
Connections:
- net +9V: now also R5.1, S1.P$7 (O)
- net GNDREF: now also J2.1, D3.1 (K), D4.1 (K), J3.R, J3.S
- net OUTPUT: now also S1.P$3 (S), S1.P$6 (S); no longer C10.2, R26.2
- net SLEEVE: no longer BT1.2 (-)
- net at J1.T: now also S1.P$2 (P)
- net at R2.1: now also S1.P$1 (O)
- net at J2.2: now also S1.P$8 (P)
- net at J2.3: now also BT1.1 (+)
- new net: J3.T, S1.P$5 (P)
- new net: BT1.2 (-), D3.2 (A)
- new net: D4.2 (A), R5.2
- new net: C10.2, R26.2, S1.P$4 (O)
- no-connect marks 12 -> 13
Other:
- moved on the sheet: BT1, C1, C3, D1, D2, J2, R1, R4, RV1

Commit message: Revision 1.0 complete.
Parts:
- removed C5: 15u, Capacitor_THT:CP_Radial_D4.0mm_P1.50mm, symbol Device:C_Polarized_Small
- removed D3: 1N914, Diode_THT:D_DO-35_SOD27_P7.62mm_Horizontal, symbol Diode:1N914
- removed Q5: 2N2219, Package_TO_SOT_THT:TO-92_Inline, symbol Transistor_BJT:2N2219
- removed R13, R24: 150K, Resistor_THT:R_Axial_DIN0207_L6.3mm_D2.5mm_P7.62mm_Horizontal, symbol Device:R_Small_US
- removed R15: 470K, Resistor_THT:R_Axial_DIN0207_L6.3mm_D2.5mm_P7.62mm_Horizontal, symbol Device:R_Small_US
- removed R4: 1M, Resistor_THT:R_Axial_DIN0207_L6.3mm_D2.5mm_P7.62mm_Horizontal, symbol Device:R_Small_US
- removed R9: 3M9, Resistor_THT:R_Axial_DIN0207_L6.3mm_D2.5mm_P7.62mm_Horizontal, symbol Device:R_Small_US
- removed RV1: 250K - Trim, symbol Device:R_Potentiometer_Trim
- removed U1, U2, U3, U4, U5, U6: TL061, Package_DIP:DIP-8_W7.62mm, symbol Amplifier_Operational:TL061
- added C11, C12: 100n, Capacitor_THT:C_Disc_D7.5mm_W2.5mm_P5.00mm, symbol Device:C_Small
- added C8: 4n7, Capacitor_THT:C_Disc_D7.5mm_W2.5mm_P5.00mm, symbol Device:C_Small
- added LFO1: STOMPLFO_DIP8, Package_DIP:DIP-8_W7.62mm_Socket, symbol ElectricDruidLFO:STOMPLFO_DIP8
- added R20: 100K, Resistor_THT:R_Axial_DIN0207_L6.3mm_D2.5mm_P10.16mm_Horizontal, symbol Device:R_Small_US
- added R21, R22: 10K, Resistor_THT:R_Axial_DIN0207_L6.3mm_D2.5mm_P10.16mm_Horizontal, symbol Device:R_Small_US
- added R26: 1K, Resistor_THT:R_Axial_DIN0207_L6.3mm_D2.5mm_P10.16mm_Horizontal, symbol Device:R_Small_US
- added R5: 150K, Resistor_THT:R_Axial_DIN0207_L6.3mm_D2.5mm_P10.16mm_Horizontal, symbol Device:R_Small_US
- added RV1, RV3: 10k, Connector_Wire:SolderWire-0.1sqmm_1x03_P3.6mm_D0.4mm_OD1mm_Relief, symbol Device:R_Potentiometer_US
- added U1: TL074, Package_DIP:DIP-14_W7.62mm, symbol Amplifier_Operational:TL074
- added U2: TL072, Package_DIP:DIP-8_W7.62mm, symbol Amplifier_Operational:TL072
- BT1: footprint Connector_JST:JST_ACH_BM02B-ACHSS-GAN-ETF_1x02-1MP_P1.20mm_Vertical -> Connector_JST:JST_EH_S2B-EH_1x02_P2.50mm_Horizontal
- C7: value 0.01u -> 47n
- D3: renamed from D2; footprint (none) -> Diode_THT:D_DO-35_SOD27_P7.62mm_Horizontal
- J1: value AudioJack3 -> InputJack; symbol Connector:AudioJack3 -> Connector:AudioJack3_Dual_Switch
- J2: renamed from J3; value AudioJack3 -> OutputJack; symbol Connector:AudioJack3 -> Connector:AudioJack3_Dual_Switch
- Q1, Q2, Q3, Q4: symbol Transistor_FET:2N7000 -> Transistor_FET:BF245A
- R1: renamed from R8; footprint Resistor_THT:R_Axial_DIN0207_L6.3mm_D2.5mm_P7.62mm_Horizontal -> Resistor_THT:R_Axial_DIN0207_L6.3mm_D2.5mm_P10.16mm_Horizontal
- R10: renamed from R22; footprint Resistor_THT:R_Axial_DIN0207_L6.3mm_D2.5mm_P7.62mm_Horizontal -> Resistor_THT:R_Axial_DIN0207_L6.3mm_D2.5mm_P10.16mm_Horizontal
- R11: renamed from R2; footprint Resistor_THT:R_Axial_DIN0207_L6.3mm_D2.5mm_P7.62mm_Horizontal -> Resistor_THT:R_Axial_DIN0207_L6.3mm_D2.5mm_P10.16mm_Horizontal
- R12: value 150K -> 500; footprint Resistor_THT:R_Axial_DIN0207_L6.3mm_D2.5mm_P7.62mm_Horizontal -> Resistor_THT:R_Axial_DIN0207_L6.3mm_D2.5mm_P10.16mm_Horizontal
- R13: renamed from R3; footprint Resistor_THT:R_Axial_DIN0207_L6.3mm_D2.5mm_P7.62mm_Horizontal -> Resistor_THT:R_Axial_DIN0207_L6.3mm_D2.5mm_P10.16mm_Horizontal
- R14: renamed from R7; footprint Resistor_THT:R_Axial_DIN0207_L6.3mm_D2.5mm_P7.62mm_Horizontal -> Resistor_THT:R_Axial_DIN0207_L6.3mm_D2.5mm_P10.16mm_Horizontal
- R15: renamed from R11; footprint Resistor_THT:R_Axial_DIN0207_L6.3mm_D2.5mm_P7.62mm_Horizontal -> Resistor_THT:R_Axial_DIN0207_L6.3mm_D2.5mm_P10.16mm_Horizontal
- R16: renamed from R17; footprint Resistor_THT:R_Axial_DIN0207_L6.3mm_D2.5mm_P7.62mm_Horizontal -> Resistor_THT:R_Axial_DIN0207_L6.3mm_D2.5mm_P10.16mm_Horizontal
- R17: renamed from R20; footprint Resistor_THT:R_Axial_DIN0207_L6.3mm_D2.5mm_P7.62mm_Horizontal -> Resistor_THT:R_Axial_DIN0207_L6.3mm_D2.5mm_P10.16mm_Horizontal
- R18: renamed from R26; footprint Resistor_THT:R_Axial_DIN0207_L6.3mm_D2.5mm_P7.62mm_Horizontal -> Resistor_THT:R_Axial_DIN0207_L6.3mm_D2.5mm_P10.16mm_Horizontal
- R19: renamed from R5; footprint Resistor_THT:R_Axial_DIN0207_L6.3mm_D2.5mm_P7.62mm_Horizontal -> Resistor_THT:R_Axial_DIN0207_L6.3mm_D2.5mm_P10.16mm_Horizontal
- R2: renamed from R14; footprint Resistor_THT:R_Axial_DIN0207_L6.3mm_D2.5mm_P7.62mm_Horizontal -> Resistor_THT:R_Axial_DIN0207_L6.3mm_D2.5mm_P10.16mm_Horizontal
- R23: value 150K -> 10K; footprint Resistor_THT:R_Axial_DIN0207_L6.3mm_D2.5mm_P7.62mm_Horizontal -> Resistor_THT:R_Axial_DIN0207_L6.3mm_D2.5mm_P10.16mm_Horizontal
- R24: renamed from R1; footprint Resistor_THT:R_Axial_DIN0207_L6.3mm_D2.5mm_P7.62mm_Horizontal -> Resistor_THT:R_Axial_DIN0207_L6.3mm_D2.5mm_P10.16mm_Horizontal
- R25: value 56K -> 1K; footprint Resistor_THT:R_Axial_DIN0207_L6.3mm_D2.5mm_P7.62mm_Horizontal -> Resistor_THT:R_Axial_DIN0207_L6.3mm_D2.5mm_P10.16mm_Horizontal
- R3: renamed from R18; footprint Resistor_THT:R_Axial_DIN0207_L6.3mm_D2.5mm_P7.62mm_Horizontal -> Resistor_THT:R_Axial_DIN0207_L6.3mm_D2.5mm_P10.16mm_Horizontal
- R4: renamed from R21; footprint Resistor_THT:R_Axial_DIN0207_L6.3mm_D2.5mm_P7.62mm_Horizontal -> Resistor_THT:R_Axial_DIN0207_L6.3mm_D2.5mm_P10.16mm_Horizontal
- R6: footprint Resistor_THT:R_Axial_DIN0207_L6.3mm_D2.5mm_P7.62mm_Horizontal -> Resistor_THT:R_Axial_DIN0207_L6.3mm_D2.5mm_P10.16mm_Horizontal
- R7: renamed from R10; footprint Resistor_THT:R_Axial_DIN0207_L6.3mm_D2.5mm_P7.62mm_Horizontal -> Resistor_THT:R_Axial_DIN0207_L6.3mm_D2.5mm_P10.16mm_Horizontal
- R8: renamed from R16; footprint Resistor_THT:R_Axial_DIN0207_L6.3mm_D2.5mm_P7.62mm_Horizontal -> Resistor_THT:R_Axial_DIN0207_L6.3mm_D2.5mm_P10.16mm_Horizontal
- R9: renamed from R19; footprint Resistor_THT:R_Axial_DIN0207_L6.3mm_D2.5mm_P7.62mm_Horizontal -> Resistor_THT:R_Axial_DIN0207_L6.3mm_D2.5mm_P10.16mm_Horizontal
- RV2: value 470K -> 10k; footprint (none) -> Connector_Wire:SolderWire-0.1sqmm_1x03_P3.6mm_D0.4mm_OD1mm_Relief
- renumbered C2 to C1, C3 to C10, C4 to C2, C6 to C3, C8 to C4, C9 to C5, C10 to C6, C1 to C9, D4 to D1, D1 to D2, J2 to J3
Connections:
- net VAA is gone; now on net +5V: R13.1
- net +5V: now also R23.1, RV2.3, LFO1.1 (+5V), RV3.3, U2.3 (+)
- net +9V: now also U1.4 (V+), U2.8 (V+)
- net GNDREF: now also C10.1, C7.1, J1.S1, J2.R1, J2.S1, RV2.1, C11.1, C12.1, C8.1, LFO1.8 (GND), R22.2, RV3.1, U1.11 (V-), U2.4 (V-); no longer J1.R, J2.R, J2.S, J3.1, R25.1
- net U1_LOOPBACK: now also RV1.1, RV1.2, U2.6 (-), U2.7; no longer R23.1
- net at S1.P$5 (P): now also J2.T1; no longer J2.T
- net at C1.2, R13.2: now also U2.5 (+)
- net at R3.1, R8.2: now also U1.9 (-)
- net at C5.1, R3.2, R9.1: now also U1.8
- net at C6.1: now also R5.2, U2.1; no longer R25.2
- net RING: now reaches BT1.2 (-)
- net RING: now also J1.R1, J3.1
- net at C3.2, R15.2: now also Q2.2 (S), U1.3 (+); no longer Q2.1 (S)
- net at C5.2, R17.2: now also Q4.2 (S), U1.12 (+); no longer Q4.1 (S)
- net at R2.1, R7.2: now also U1.2 (-)
- net at C4.1, R2.2, R8.1: now also U1.1
- net at S1.P$2 (P): now also J1.T1; no longer J1.T
- net at R4.1, R9.2: now also U1.13 (-)
- net at R10.1, R4.2: now also U1.14
- net at C3.1, R1.2, R7.1: now also U1.7
- net at R12.1: now also S1.P$4 (O); no longer C7.1
- net LFO_OUT: now reaches C7.2
- net LFO_OUT: now also Q1.1 (G), Q2.1 (G), Q3.1 (G), Q4.1 (G), R20.2; no longer RV2.3
- net at C4.2, R16.2: now also Q3.2 (S), U1.10 (+); no longer Q3.1 (S)
- net at C6.2, R18.2: now also R12.2; no longer S1.P$4 (O)
- net at R1.1, R6.2: now also U1.6 (-)
- net at C2.2, R14.2: now also Q1.2 (S), U1.5 (+); no longer Q1.1 (S)
- net at R23.2: now also LFO1.5 (DPTH); no longer R10.2
- removed net SLEEVE: J1.S
- removed net VDD: C10.1, Q1.2 (G), Q2.2 (G), Q3.2 (G), Q4.2 (G)
- new net: C8.2, R20.1, R21.2
- new net: LFO1.2 (OFFST), R22.1
- new net: R26.1, RV3.2
- new net: R10.2, R5.1, RV1.3, U2.2 (-)
- new net: R25.1, RV2.2
- new net FRQ: C11.2, LFO1.7 (FRQ), R25.2
- new net LFO: LFO1.3 (OUT), R21.1
- new net WVF: C12.2, LFO1.6 (WVF), R26.2
- no-connect marks 13 -> 8
Other:
- note added: "INPUT BUFFER"
- note added: "LOW FREQUENCY OSCILLATOR WITH CONTROLS"
- note added: "MIXING STAGE"
- note added: "PHASING STAGES"
- note added: "POWER CONDITIONING, SWITCHING, AND INDICATOR"
- note removed: "TODO: ADD POLARITY PROTECTION, MAYBE AN INDICATOR LED ALSO FIX THE BATTERY SWITCHING CIRCUIT"
- company: (none) -> Lord & Murphy
- title: (none) -> Half-Pi++
- moved on the sheet: BT1, C1, C10, C2, C3, C4, C5, C6, C9, D1, D2, D3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
